Commit message: First implementation of Gazebo sim, sensor fusion packages, and Ignition migration
- Migrate wheelchair description package from CAD_MODELS to thesis_ws/src/gazebo
- Add Ignition Gazebo simulation with diff-drive controller and LiDAR sensors
- Switch LiDAR sensor type to gpu_lidar and bridge topics to ignition.msgs namespace
- Fix wheelchair spawn orientation (roll = 1.5708 rad)
- Add lidar_camera_fusion_pcl and lidar_camera_object_association ROS2 packages
- Add submodule pointers for rslidar_sdk, rslidar_msg, and zed-ros2-wrapper
- Add TimestampsCorrector.py and convert.yaml for bag post-processing
- Update .gitignore to exclude large ROS bag files (*.db3) and build artifacts

Co-Authored-By: Claude Sonnet 4.6 <noreply@anthropic.com>

File: thesis_ws/src/gazebo/wheelchair_actual_set_up_description/urdf/materials.xacro (robot description, xacro)
@@ -1,4 +1,4 @@
 <?xml version="1.0" ?>
-<robot name="Wheelchair_ActualSetUp" xmlns:xacro="http://www.ros.org/wiki/xacro" >
+<robot name="wheelchair_actual_set_up" xmlns:xacro="http://www.ros.org/wiki/xacro" >
 <material name="silver">
   <color rgba="0.700 0.700 0.700 1.000"/>

File: thesis_ws/src/gazebo/wheelchair_actual_set_up_description/urdf/wheelchair_actual_set_up.xacro (robot description, xacro)
@@ -1,7 +1,7 @@
 <?xml version="1.0" ?>
-<robot name="Wheelchair_ActualSetUp" xmlns:xacro="http://www.ros.org/wiki/xacro">
-<xacro:include filename="$(find Wheelchair_ActualSetUp_description)/urdf/materials.xacro" />
-<xacro:include filename="$(find Wheelchair_ActualSetUp_description)/urdf/Wheelchair_ActualSetUp.trans" />
-<xacro:include filename="$(find Wheelchair_ActualSetUp_description)/urdf/Wheelchair_ActualSetUp.gazebo" />
+<robot name="wheelchair_actual_set_up" xmlns:xacro="http://www.ros.org/wiki/xacro">
+<xacro:include filename="$(find wheelchair_actual_set_up_description)/urdf/materials.xacro" />
+<xacro:include filename="$(find wheelchair_actual_set_up_description)/urdf/wheelchair_actual_set_up.trans" />
+<xacro:include filename="$(find wheelchair_actual_set_up_description)/urdf/wheelchair_actual_set_up.gazebo" />
 <link name="base_link">
   <inertial>
@@ -13,5 +13,5 @@
     <origin xyz="0 0 0" rpy="0 0 0"/>
     <geometry>
-      <mesh filename="package://Wheelchair_ActualSetUp_description/meshes/base_link.stl" scale="0.001 0.001 0.001"/>
+      <mesh filename="package://wheelchair_actual_set_up_description/meshes/base_link.stl" scale="0.001 0.001 0.001"/>
     </geometry>
     <material name="silver"/>
@@ -20,5 +20,5 @@
     <origin xyz="0 0 0" rpy="0 0 0"/>
     <geometry>
-      <mesh filename="package://Wheelchair_ActualSetUp_description/meshes/base_link.stl" scale="0.001 0.001 0.001"/>
+      <mesh filename="package://wheelchair_actual_set_up_description/meshes/base_link.stl" scale="0.001 0.001 0.001"/>
     </geometry>
   </collision>
@@ -33,5 +33,5 @@
     <origin xyz="-0.24 -0.175 -0.205" rpy="0 0 0"/>
     <geometry>
-      <mesh filename="package://Wheelchair_ActualSetUp_description/meshes/left_Wheel_1.stl" scale="0.001 0.001 0.001"/>
+      <mesh filename="package://wheelchair_actual_set_up_description/meshes/left_Wheel_1.stl" scale="0.001 0.001 0.001"/>
     </geometry>
     <material name="silver"/>
@@ -40,5 +40,5 @@
     <origin xyz="-0.24 -0.175 -0.205" rpy="0 0 0"/>
     <geometry>
-      <mesh filename="package://Wheelchair_ActualSetUp_description/meshes/left_Wheel_1.stl" scale="0.001 0.001 0.001"/>
+      <mesh filename="package://wheelchair_actual_set_up_description/meshes/left_Wheel_1.stl" scale="0.001 0.001 0.001"/>
     </geometry>
   </collision>
@@ -53,5 +53,5 @@
     <origin xyz="0.24 -0.175 -0.205" rpy="0 0 0"/>
     <geometry>
-      <mesh filename="package://Wheelchair_ActualSetUp_description/meshes/right_Wheel_1.stl" scale="0.001 0.001 0.001"/>
+      <mesh filename="package://wheelchair_actual_set_up_description/meshes/right_Wheel_1.stl" scale="0.001 0.001 0.001"/>
     </geometry>
     <material name="silver"/>
@@ -60,5 +60,5 @@
     <origin xyz="0.24 -0.175 -0.205" rpy="0 0 0"/>
     <geometry>
-      <mesh filename="package://Wheelchair_ActualSetUp_description/meshes/right_Wheel_1.stl" scale="0.001 0.001 0.001"/>
+      <mesh filename="package://wheelchair_actual_set_up_description/meshes/right_Wheel_1.stl" scale="0.001 0.001 0.001"/>
     </geometry>
   </collision>
@@ -73,5 +73,5 @@
     <origin xyz="0.28 -0.28 -0.65" rpy="0 0 0"/>
     <geometry>
-      <mesh filename="package://Wheelchair_ActualSetUp_description/meshes/right_caster_support_1.stl" scale="0.001 0.001 0.001"/>
+      <mesh filename="package://wheelchair_actual_set_up_description/meshes/right_caster_support_1.stl" scale="0.001 0.001 0.001"/>
     </geometry>
     <material name="silver"/>
@@ -80,5 +80,5 @@
     <origin xyz="0.28 -0.28 -0.65" rpy="0 0 0"/>
     <geometry>
-      <mesh filename="package://Wheelchair_ActualSetUp_description/meshes/right_caster_support_1.stl" scale="0.001 0.001 0.001"/>
+      <mesh filename="package://wheelchair_actual_set_up_description/meshes/right_caster_support_1.stl" scale="0.001 0.001 0.001"/>
     </geometry>
   </collision>
@@ -93,5 +93,5 @@
     <origin xyz="0.2875 -0.075 -0.705003" rpy="0 0 0"/>
     <geometry>
-      <mesh filename="package://Wheelchair_ActualSetUp_description/meshes/right_caster_2_1.stl" scale="0.001 0.001 0.001"/>
+      <mesh filename="package://wheelchair_actual_set_up_description/meshes/right_caster_2_1.stl" scale="0.001 0.001 0.001"/>
     </geometry>
     <material name="silver"/>
@@ -100,5 +100,5 @@
     <origin xyz="0.2875 -0.075 -0.705003" rpy="0 0 0"/>
     <geometry>
-      <mesh filename="package://Wheelchair_ActualSetUp_description/meshes/right_caster_2_1.stl" scale="0.001 0.001 0.001"/>
+      <mesh filename="package://wheelchair_actual_set_up_description/meshes/right_caster_2_1.stl" scale="0.001 0.001 0.001"/>
     </geometry>
   </collision>
@@ -113,5 +113,5 @@
     <origin xyz="0.2725 -0.075 -0.705003" rpy="0 0 0"/>
     <geometry>
-      <mesh filename="package://Wheelchair_ActualSetUp_description/meshes/right_caster_1_1.stl" scale="0.001 0.001 0.001"/>
+      <mesh filename="package://wheelchair_actual_set_up_description/meshes/right_caster_1_1.stl" scale="0.001 0.001 0.001"/>
     </geometry>
     <material name="silver"/>
@@ -120,5 +120,5 @@
     <origin xyz="0.2725 -0.075 -0.705003" rpy="0 0 0"/>
     <geometry>
-      <mesh filename="package://Wheelchair_ActualSetUp_description/meshes/right_caster_1_1.stl" scale="0.001 0.001 0.001"/>
+      <mesh filename="package://wheelchair_actual_set_up_description/meshes/right_caster_1_1.stl" scale="0.001 0.001 0.001"/>
     </geometry>
   </collision>
@@ -133,5 +133,5 @@
     <origin xyz="-0.28 -0.28 -0.65" rpy="0 0 0"/>
     <geometry>
-      <mesh filename="package://Wheelchair_ActualSetUp_description/meshes/left_caster_support_1.stl" scale="0.001 0.001 0.001"/>
+      <mesh filename="package://wheelchair_actual_set_up_description/meshes/left_caster_support_1.stl" scale="0.001 0.001 0.001"/>
     </geometry>
     <material name="silver"/>
@@ -140,5 +140,5 @@
     <origin xyz="-0.28 -0.28 -0.65" rpy="0 0 0"/>
     <geometry>
-      <mesh filename="package://Wheelchair_ActualSetUp_description/meshes/left_caster_support_1.stl" scale="0.001 0.001 0.001"/>
+      <mesh filename="package://wheelchair_actual_set_up_description/meshes/left_caster_support_1.stl" scale="0.001 0.001 0.001"/>
     </geometry>
   </collision>
@@ -153,5 +153,5 @@
     <origin xyz="-0.2725 -0.075 -0.705003" rpy="0 0 0"/>
     <geometry>
-      <mesh filename="package://Wheelchair_ActualSetUp_description/meshes/left_caster_1_1.stl" scale="0.001 0.001 0.001"/>
+      <mesh filename="package://wheelchair_actual_set_up_description/meshes/left_caster_1_1.stl" scale="0.001 0.001 0.001"/>
     </geometry>
     <material name="silver"/>
@@ -160,5 +160,5 @@
     <origin xyz="-0.2725 -0.075 -0.705003" rpy="0 0 0"/>
     <geometry>
-      <mesh filename="package://Wheelchair_ActualSetUp_description/meshes/left_caster_1_1.stl" scale="0.001 0.001 0.001"/>
+      <mesh filename="package://wheelchair_actual_set_up_description/meshes/left_caster_1_1.stl" scale="0.001 0.001 0.001"/>
     </geometry>
   </collision>
@@ -173,5 +173,5 @@
     <origin xyz="-0.2875 -0.075 -0.705003" rpy="0 0 0"/>
     <geometry>
-      <mesh filename="package://Wheelchair_ActualSetUp_description/meshes/left_caster_2_1.stl" scale="0.001 0.001 0.001"/>
+      <mesh filename="package://wheelchair_actual_set_up_description/meshes/left_caster_2_1.stl" scale="0.001 0.001 0.001"/>
     </geometry>
     <material name="silver"/>
@@ -180,5 +180,5 @@
     <origin xyz="-0.2875 -0.075 -0.705003" rpy="0 0 0"/>
     <geometry>
-      <mesh filename="package://Wheelchair_ActualSetUp_description/meshes/left_caster_2_1.stl" scale="0.001 0.001 0.001"/>
+      <mesh filename="package://wheelchair_actual_set_up_description/meshes/left_caster_2_1.stl" scale="0.001 0.001 0.001"/>
     </geometry>
   </collision>
@@ -193,5 +193,5 @@
     <origin xyz="0.168 -0.05 0.0175" rpy="0 0 0"/>
     <geometry>
-      <mesh filename="package://Wheelchair_ActualSetUp_description/meshes/rear_caster_4_1.stl" scale="0.001 0.001 0.001"/>
+      <mesh filename="package://wheelchair_actual_set_up_description/meshes/rear_caster_4_1.stl" scale="0.001 0.001 0.001"/>
     </geometry>
     <material name="silver"/>
@@ -200,5 +200,5 @@
     <origin xyz="0.168 -0.05 0.0175" rpy="0 0 0"/>
     <geometry>
-      <mesh filename="package://Wheelchair_ActualSetUp_description/meshes/rear_caster_4_1.stl" scale="0.001 0.001 0.001"/>
+      <mesh filename="package://wheelchair_actual_set_up_description/meshes/rear_caster_4_1.stl" scale="0.001 0.001 0.001"/>
     </geometry>
   </collision>
@@ -213,5 +213,5 @@
     <origin xyz="-0.168 -0.05 0.0175" rpy="0 0 0"/>
     <geometry>
-      <mesh filename="package://Wheelchair_ActualSetUp_description/meshes/rear_caster_3_1.stl" scale="0.001 0.001 0.001"/>
+      <mesh filename="package://wheelchair_actual_set_up_description/meshes/rear_caster_3_1.stl" scale="0.001 0.001 0.001"/>
     </geometry>
     <material name="silver"/>
@@ -220,5 +220,5 @@
     <origin xyz="-0.168 -0.05 0.0175" rpy="0 0 0"/>
     <geometry>
-      <mesh filename="package://Wheelchair_ActualSetUp_description/meshes/rear_caster_3_1.stl" scale="0.001 0.001 0.001"/>
+      <mesh filename="package://wheelchair_actual_set_up_description/meshes/rear_caster_3_1.stl" scale="0.001 0.001 0.001"/>
     </geometry>
   </collision>
@@ -233,5 +233,5 @@
     <origin xyz="0.0 -0.16 0.08" rpy="0 0 0"/>
     <geometry>
-      <mesh filename="package://Wheelchair_ActualSetUp_description/meshes/rear_caster_support_1.stl" scale="0.001 0.001 0.001"/>
+      <mesh filename="package://wheelchair_actual_set_up_description/meshes/rear_caster_support_1.stl" scale="0.001 0.001 0.001"/>
     </geometry>
     <material name="silver"/>
@@ -240,5 +240,5 @@
     <origin xyz="0.0 -0.16 0.08" rpy="0 0 0"/>
     <geometry>
-      <mesh filename="package://Wheelchair_ActualSetUp_description/meshes/rear_caster_support_1.stl" scale="0.001 0.001 0.001"/>
+      <mesh filename="package://wheelchair_actual_set_up_description/meshes/rear_caster_support_1.stl" scale="0.001 0.001 0.001"/>
     </geometry>
   </collision>
@@ -253,5 +253,5 @@
     <origin xyz="-0.0075 -0.075 0.055" rpy="0 0 0"/>
     <geometry>
-      <mesh filename="package://Wheelchair_ActualSetUp_description/meshes/rear_caster_1_1.stl" scale="0.001 0.001 0.001"/>
+      <mesh filename="package://wheelchair_actual_set_up_description/meshes/rear_caster_1_1.stl" scale="0.001 0.001 0.001"/>
     </geometry>
     <material name="silver"/>
@@ -260,5 +260,5 @@
     <origin xyz="-0.0075 -0.075 0.055" rpy="0 0 0"/>
     <geometry>
-      <mesh filename="package://Wheelchair_ActualSetUp_description/meshes/rear_caster_1_1.stl" scale="0.001 0.001 0.001"/>
+      <mesh filename="package://wheelchair_actual_set_up_description/meshes/rear_caster_1_1.stl" scale="0.001 0.001 0.001"/>
     </geometry>
   </collision>
@@ -273,5 +273,5 @@
     <origin xyz="0.0075 -0.075 0.055" rpy="0 0 0"/>
     <geometry>
-      <mesh filename="package://Wheelchair_ActualSetUp_description/meshes/rear_caster_2_1.stl" scale="0.001 0.001 0.001"/>
+      <mesh filename="package://wheelchair_actual_set_up_description/meshes/rear_caster_2_1.stl" scale="0.001 0.001 0.001"/>
     </geometry>
     <material name="silver"/>
@@ -280,5 +280,5 @@
     <origin xyz="0.0075 -0.075 0.055" rpy="0 0 0"/>
     <geometry>
-      <mesh filename="package://Wheelchair_ActualSetUp_description/meshes/rear_caster_2_1.stl" scale="0.001 0.001 0.001"/>
+      <mesh filename="package://wheelchair_actual_set_up_description/meshes/rear_caster_2_1.stl" scale="0.001 0.001 0.001"/>
     </geometry>
   </collision>
@@ -293,5 +293,5 @@
     <origin xyz="0.250052 -0.358 0.030052" rpy="0 0 0"/>
     <geometry>
-      <mesh filename="package://Wheelchair_ActualSetUp_description/meshes/rear_lidar_1.stl" scale="0.001 0.001 0.001"/>
+      <mesh filename="package://wheelchair_actual_set_up_description/meshes/rear_lidar_1.stl" scale="0.001 0.001 0.001"/>
     </geometry>
     <material name="silver"/>
@@ -300,5 +300,5 @@
     <origin xyz="0.250052 -0.358 0.030052" rpy="0 0 0"/>
     <geometry>
-      <mesh filename="package://Wheelchair_ActualSetUp_description/meshes/rear_lidar_1.stl" scale="0.001 0.001 0.001"/>
+      <mesh filename="package://wheelchair_actual_set_up_description/meshes/rear_lidar_1.stl" scale="0.001 0.001 0.001"/>
     </geometry>
   </collision>
@@ -313,5 +313,5 @@
     <origin xyz="-0.220052 -0.308 -0.760052" rpy="0 0 0"/>
     <geometry>
-      <mesh filename="package://Wheelchair_ActualSetUp_description/meshes/front_Lidar_1.stl" scale="0.001 0.001 0.001"/>
+      <mesh filename="package://wheelchair_actual_set_up_description/meshes/front_Lidar_1.stl" scale="0.001 0.001 0.001"/>
     </geometry>
     <material name="silver"/>
@@ -320,9 +320,9 @@
     <origin xyz="-0.220052 -0.308 -0.760052" rpy="0 0 0"/>
     <geometry>
-      <mesh filename="package://Wheelchair_ActualSetUp_description/meshes/front_Lidar_1.stl" scale="0.001 0.001 0.001"/>
-    </geometry>
-  </collision>
-</link>
-<joint name="Revolute 1" type="continuous">
+      <mesh filename="package://wheelchair_actual_set_up_description/meshes/front_Lidar_1.stl" scale="0.001 0.001 0.001"/>
+    </geometry>
+  </collision>
+</link>
+<joint name="left_wheel_joint" type="continuous">
   <origin xyz="0.24 0.175 0.205" rpy="0 0 0"/>
   <parent link="base_link"/>
@@ -330,5 +330,5 @@
   <axis xyz="1.0 0.0 0.0"/>
 </joint>
-<joint name="Revolute 2" type="continuous">
+<joint name="right_wheel_joint" type="continuous">
   <origin xyz="-0.24 0.175 0.205" rpy="0 0 0"/>
   <parent link="base_link"/>
@@ -336,5 +336,5 @@
   <axis xyz="-1.0 0.0 0.0"/>
 </joint>
-<joint name="Revolute 3" type="continuous">
+<joint name="right_caster_support_joint" type="continuous">
   <origin xyz="-0.28 0.28 0.65" rpy="0 0 0"/>
   <parent link="base_link"/>
@@ -342,5 +342,5 @@
   <axis xyz="0.0 -1.0 0.0"/>
 </joint>
-<joint name="Revolute 4" type="continuous">
+<joint name="right_caster_wheel_2_joint" type="continuous">
   <origin xyz="-0.0075 -0.205 0.055003" rpy="0 0 0"/>
   <parent link="right_caster_support_1"/>
@@ -348,5 +348,5 @@
   <axis xyz="1.0 0.0 0.0"/>
 </joint>
-<joint name="Revolute 5" type="continuous">
+<joint name="right_caster_wheel_1_joint" type="continuous">
   <origin xyz="0.0075 -0.205 0.055003" rpy="0 0 0"/>
   <parent link="right_caster_support_1"/>
@@ -354,5 +354,5 @@
   <axis xyz="1.0 0.0 0.0"/>
 </joint>
-<joint name="Revolute 6" type="continuous">
+<joint name="left_caster_support_joint" type="continuous">
   <origin xyz="0.28 0.28 0.65" rpy="0 0 0"/>
   <parent link="base_link"/>
@@ -360,5 +360,5 @@
   <axis xyz="0.0 -1.0 0.0"/>
 </joint>
-<joint name="Revolute 7" type="continuous">
+<joint name="left_caster_wheel_1_joint" type="continuous">
   <origin xyz="-0.0075 -0.205 0.055003" rpy="0 0 0"/>
   <parent link="left_caster_support_1"/>
@@ -366,5 +366,5 @@
   <axis xyz="-1.0 0.0 0.0"/>
 </joint>
-<joint name="Revolute 8" type="continuous">
+<joint name="left_caster_wheel_2_joint" type="continuous">
   <origin xyz="0.0075 -0.205 0.055003" rpy="0 0 0"/>
   <parent link="left_caster_support_1"/>
@@ -372,5 +372,5 @@
   <axis xyz="1.0 0.0 0.0"/>
 </joint>
-<joint name="Revolute 9" type="continuous">
+<joint name="rear_caster_wheel_4_joint" type="continuous">
   <origin xyz="-0.168 0.05 -0.0175" rpy="0 0 0"/>
   <parent link="base_link"/>
@@ -378,5 +378,5 @@
   <axis xyz="1.0 0.0 0.0"/>
 </joint>
-<joint name="Revolute 10" type="continuous">
+<joint name="rear_caster_wheel_3_joint" type="continuous">
   <origin xyz="0.168 0.05 -0.0175" rpy="0 0 0"/>
   <parent link="base_link"/>
@@ -384,5 +384,5 @@
   <axis xyz="-1.0 0.0 0.0"/>
 </joint>
-<joint name="Revolute 11" type="continuous">
+<joint name="rear_caster_support_joint" type="continuous">
   <origin xyz="0.0 0.16 -0.08" rpy="0 0 0"/>
   <parent link="base_link"/>
@@ -390,5 +390,5 @@
   <axis xyz="0.0 -1.0 0.0"/>
 </joint>
-<joint name="Revolute 12" type="continuous">
+<joint name="rear_caster_wheel_1_joint" type="continuous">
   <origin xyz="0.0075 -0.085 0.025" rpy="0 0 0"/>
   <parent link="rear_caster_support_1"/>
@@ -396,5 +396,5 @@
   <axis xyz="1.0 0.0 0.0"/>
 </joint>
-<joint name="Revolute 13" type="continuous">
+<joint name="rear_caster_wheel_2_joint" type="continuous">
   <origin xyz="-0.0075 -0.085 0.025" rpy="0 0 0"/>
   <parent link="rear_caster_support_1"/>
@@ -402,13 +402,28 @@
   <axis xyz="-1.0 0.0 0.0"/>
 </joint>
-<joint name="Rigid 14" type="fixed">
+<joint name="rear_lidar_joint" type="fixed">
   <origin xyz="-0.250052 0.358 -0.030052" rpy="0 0 0"/>
   <parent link="base_link"/>
   <child link="rear_lidar_1"/>
 </joint>
-<joint name="Rigid 15" type="fixed">
+<joint name="front_lidar_joint" type="fixed">
   <origin xyz="0.220052 0.308 0.760052" rpy="0 0 0"/>
   <parent link="base_link"/>
   <child link="front_Lidar_1"/>
 </joint>
+<ros2_control name="WheelchairSystem" type="system">
+  <hardware>
+    <plugin>gz_ros2_control/GazeboSimSystem</plugin>
+  </hardware>
+  <joint name="left_wheel_joint">
+    <command_interface name="velocity"/>
+    <state_interface name="velocity"/>
+    <state_interface name="position"/>
+  </joint>
+  <joint name="right_wheel_joint">
+    <command_interface name="velocity"/>
+    <state_interface name="velocity"/>
+    <state_interface name="position"/>
+  </joint>
+</ros2_control>
 </robot>
